Commit message: ik issue: joint limit

File: pybullet_robot_envs/panda_envs/robot_data/franka_panda/panda_model.urdf (robot description, URDF)
Before this commit: robot panda, 13 links, 12 joints
Joints:
- joint panda_joint7: origin xyz=0.088 0 0 rpy=1.57079632679 0 0 -> xyz=0.088 0.107 0 rpy=1.57079632679 0 0
